File: TSOC_Teensy3x/TSOC_Teensy3X.brd (EAGLE design)
At the start: 44.5 x 30.5 mm, 14 parts, among them J1 4P-2.0, J2 4P-2.0

Commit message: update to R1.1
Parts:
- removed 5V0: JMP-2-NC, PatternAgents-ProtoPads:JMP-2-NC
- moved 3V3 0.57 mm to (39.9, 4.06)
Connections:
- removed net RXD: TEENSY.1, TSOC.7C
- removed net TXD: TEENSY.0, TSOC.8C
- removed net VIN: 5V0.1, TEENSY.VIN
- new net RXD1: TEENSY.0, TSOC.7C
- new net TXD1: TEENSY.1, TSOC.8C
- net 5V0: now also TEENSY.VIN; no longer 5V0.2
Routing:
- net TXD: track 41.2 -> 0.00 mm, vias 2 -> 0
- net RXD1: track 0.00 -> 38.6 mm, vias 0 -> 2
- net TXD1: track 0.00 -> 37.7 mm, vias 0 -> 2
- net RXD: track 36.1 -> 0.00 mm, vias 2 -> 0
- net GND: track 125.1 -> 99.7 mm, vias 7 -> 5
- net VIN: track 2.81 -> 0.00 mm
- net 3V3: track 76.3 -> 77.3 mm
- net 5V0: track 34.6 -> 34.0 mm, vias 1 -> 0
Other:
- board text added: "Rev. 1.1"
- board text removed: "Rev. 1.0"
