File: TSOC_Teensy3x/TSOC_Teensy3X.brd (EAGLE design)
At the start: 49.5 x 30.5 mm, 12 parts, among them J1 4P-2.0-90D, J2 4P-2.0-90D, J3 4P-2.0-90D

Commit message: update documentation
Connections:
- net !ATN renamed D6
- net !CS renamed D10
- net !CTS renamed A2
- net !DCD renamed A8
- net !DSR renamed A7
- net !DTR renamed A3
- net !IRQ renamed A1
- net !RI renamed A9
- net !RTS renamed A6
- net IO1 renamed D3
- net IO2 renamed D2
- net MISO renamed D11
- net MOSI renamed D12
- net RXD1 renamed D0
- net RXD3 renamed D7
- net SCK renamed D13
- net SCL renamed A5
- net SDA renamed A4
- net SS1 renamed D5
- net SS2 renamed D4
- net TXD1 renamed D1
- net TXD3 renamed D8
Changed lines of the file:
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@@
 <wire x1="39.576" y1="11.986" x2="39.624" y2="11.938" width="0.8128" layer="16"/>
 </signal>
-<signal name="!ATN">
+<signal name="D6">
 <contactref element="TSOC" pad="6B"/>
 <contactref element="TEENSY" pad="6"/>
 <wire x1="24.384" y1="26.67" x2="24.384" y2="22.86" width="0.254" layer="16"/>
 </signal>
-<signal name="SCL">
+<signal name="A5">
 <contactref element="TEENSY" pad="19/A5"/>
 <wire x1="16.764" y1="3.81" x2="15.494" y2="5.08" width="0.254" layer="1"/>
@@
 <wire x1="15.494" y1="13.716" x2="15.494" y2="10.414" width="0.254" layer="16"/>
 </signal>
-<signal name="SDA">
+<signal name="A4">
 <contactref element="TEENSY" pad="18/A4"/>
 <wire x1="14.224" y1="3.81" x2="12.954" y2="5.08" width="0.254" layer="1"/>
@@
 <wire x1="12.446" y1="8.89" x2="12.954" y2="9.398" width="0.254" layer="16"/>
 </signal>
-<signal name="SCK">
+<signal name="D13">
 <contactref element="TEENSY" pad="13"/>
 <wire x1="18.034" y1="19.05" x2="18.034" y2="25.4" width="0.254" layer="1"/>
@@
 <via x="18.034" y="19.05" extent="1-16" drill="0.3556"/>
 </signal>
-<signal name="MISO">
+<signal name="D11">
 <contactref element="TEENSY" pad="11"/>
 <wire x1="11.684" y1="22.86" x2="11.684" y2="23.114" width="0.254" layer="16"/>
@@
 <contactref element="TSOC" pad="9B"/>
 </signal>
-<signal name="MOSI">
+<signal name="D12">
 <contactref element="TEENSY" pad="12"/>
 <wire x1="9.144" y1="22.86" x2="9.144" y2="24.13" width="0.254" layer="16"/>
@@
 <contactref element="TSOC" pad="10B"/>
 </signal>
-<signal name="!CS">
+<signal name="D10">
 <contactref element="TEENSY" pad="10"/>
 <wire x1="14.224" y1="22.86" x2="16.256" y2="24.892" width="0.254" layer="16"/>
@@
 <contactref element="TSOC" pad="7B"/>
 </signal>
-<signal name="SS2">
+<signal name="D4">
 <contactref element="TEENSY" pad="4"/>
 <wire x1="29.464" y1="22.86" x2="29.464" y2="24.13" width="0.254" layer="16"/>
@@
 <contactref element="TSOC" pad="3B"/>
 </signal>
-<signal name="SS1">
+<signal name="D5">
 <contactref element="TEENSY" pad="5"/>
 <wire x1="26.924" y1="22.86" x2="26.924" y2="24.13" width="0.254" layer="16"/>
@@
 <contactref element="TSOC" pad="4B"/>
 </signal>
-<signal name="IO2">
+<signal name="D2">
 <contactref element="TEENSY" pad="2"/>
 <wire x1="34.544" y1="22.86" x2="34.544" y2="24.13" width="0.254" layer="16"/>
@@
 <contactref element="TSOC" pad="1B"/>
 </signal>
-<signal name="IO1">
+<signal name="D3">
 <contactref element="TEENSY" pad="3"/>
 <wire x1="32.004" y1="22.86" x2="32.004" y2="24.13" width="0.254" layer="16"/>
@@
 <contactref element="TSOC" pad="2B"/>
 </signal>
-<signal name="!IRQ">
+<signal name="A1">
 <contactref element="TSOC" pad="5B"/>
 <contactref element="TEENSY" pad="15/A1"/>
@@
 <wire x1="28.194" y1="25.4" x2="26.924" y2="26.67" width="0.254" layer="1"/>
 </signal>
-<signal name="!RTS">
+<signal name="A6">
 <contactref element="TSOC" pad="5C"/>
 <contactref element="TEENSY" pad="20/A6"/>
 <wire x1="26.924" y1="7.62" x2="26.924" y2="3.81" width="0.254" layer="1"/>
 </signal>
-<signal name="!CTS">
+<signal name="A2">
 <contactref element="TEENSY" pad="16/A2"/>
 <wire x1="16.764" y1="7.62" x2="16.764" y2="11.43" width="0.254" layer="1"/>
@@
 <contactref element="TSOC" pad="6C"/>
 </signal>
-<signal name="!RI">
+<signal name="A9">
 <contactref element="TEENSY" pad="23/A9"/>
 <wire x1="37.084" y1="3.81" x2="37.084" y2="5.08" width="0.254" layer="1"/>
@@
 <contactref element="TSOC" pad="1C"/>
 </signal>
-<signal name="!DCD">
+<signal name="A8">
 <contactref element="TEENSY" pad="22/A8"/>
 <wire x1="34.544" y1="3.81" x2="34.544" y2="5.08" width="0.254" layer="1"/>
@@
 <contactref element="TSOC" pad="2C"/>
 </signal>
-<signal name="!DSR">
+<signal name="A7">
 <contactref element="TEENSY" pad="21/A7"/>
 <wire x1="32.004" y1="3.81" x2="32.004" y2="5.08" width="0.254" layer="1"/>
@@
 <contactref element="TSOC" pad="3C"/>
 </signal>
-<signal name="!DTR">
+<signal name="A3">
 <contactref element="TSOC" pad="4C"/>
 <contactref element="TEENSY" pad="17/A3"/>
@@
 <wire x1="37.084" y1="9.652" x2="37.084" y2="7.62" width="0.8128" layer="16"/>
 </signal>
-<signal name="RXD3">
+<signal name="D7">
 <contactref element="TEENSY" pad="7"/>
 <contactref element="J2" pad="1"/>
@@
 <wire x1="21.844" y1="20.574" x2="21.844" y2="22.86" width="0.254" layer="16"/>
 </signal>
-<signal name="TXD3">
+<signal name="D8">
 <contactref element="TEENSY" pad="8"/>
 <contactref element="J2" pad="2"/>
@@
 <wire x1="19.304" y1="22.098" x2="19.304" y2="22.86" width="0.254" layer="16"/>
 </signal>
-<signal name="RXD1">
+<signal name="D0">
 <contactref element="TEENSY" pad="0"/>
 <via x="30.734" y="19.05" extent="1-16" drill="0.3556"/>
@@
 <wire x1="37.592" y1="20.828" x2="39.624" y2="22.86" width="0.254" layer="1"/>
 </signal>
-<signal name="TXD1">
+<signal name="D1">
 <contactref element="TEENSY" pad="1"/>
 <via x="29.718" y="15.24" extent="1-16" drill="0.3556"/>
