File: TSOC_Teensy3x/TSOC_Teensy3X.sch (EAGLE design)
At the start: 13 parts, among them J1 4P-2.0, J2 4P-2.0

Commit message: update to R1.1
Parts:
- removed 5V0: JMP-2-NC, PatternAgents-ProtoPads:JMP-2-NC
Connections:
- removed net RXD: TEENSY.1, TSOC.RXD
- removed net TXD: TEENSY.0, TSOC.TXD
- removed net VIN: 5V0.1, TEENSY.VIN
- new net RXD1: TEENSY.0, TSOC.RXD
- new net TXD1: TEENSY.1, TSOC.TXD
- net 5V0: now also TEENSY.VIN; no longer 5V0.2
