File: TSOC_Teensy3x/TSOC_Teensy3X.sch (EAGLE design)
At the start: 11 parts, among them J1 4P-2.0-90D, J2 4P-2.0-90D, J3 4P-2.0-90D

Commit message: update documentation
Connections:
- net !ATN renamed D6
- net !CS renamed D10
- net !CTS renamed A2
- net !DCD renamed A8
- net !DSR renamed A7
- net !DTR renamed A3
- net !IRQ renamed A1
- net !RI renamed A9
- net !RTS renamed A6
- net IO1 renamed D3
- net IO2 renamed D2
- net MISO renamed D11
- net MOSI renamed D12
- net RXD1 renamed D0
- net RXD3 renamed D7
- net SCK renamed D13
- net SCL renamed A5
- net SDA renamed A4
- net SS1 renamed D5
- net SS2 renamed D4
- net TXD1 renamed D1
- net TXD3 renamed D8
Changed lines of the file:
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@@
 <setting verticaltext="up"/>
 </settings>
-<grid distance="0.05" unitdist="inch" unit="inch" style="dots" multiple="1" display="yes" altdistance="0.01" altunitdist="inch" altunit="inch"/>
+<grid distance="0.1" unitdist="inch" unit="inch" style="lines" multiple="1" display="no" altdistance="0.01" altunitdist="inch" altunit="inch"/>
 <layers>
 <layer number="1" name="Top" color="4" fill="1" visible="no" active="no"/>
@@
 </segment>
 </net>
-<net name="!ATN" class="0">
+<net name="D6" class="0">
 <segment>
 <wire x1="129.54" y1="78.74" x2="134.62" y2="78.74" width="0.1524" layer="91"/>
@@
 </segment>
 </net>
-<net name="SCL" class="0">
+<net name="A5" class="0">
 <segment>
 <pinref part="TEENSY" gate="G$1" pin="19/A5"/>
@@
 </segment>
 </net>
-<net name="SDA" class="0">
+<net name="A4" class="0">
 <segment>
 <pinref part="TEENSY" gate="G$1" pin="18/A4"/>
@@
 </segment>
 </net>
-<net name="SCK" class="0">
+<net name="D13" class="0">
 <segment>
 <wire x1="129.54" y1="101.6" x2="134.62" y2="101.6" width="0.1524" layer="91"/>
@@
 </segment>
 </net>
-<net name="MISO" class="0">
+<net name="D11" class="0">
 <segment>
 <wire x1="129.54" y1="99.06" x2="134.62" y2="99.06" width="0.1524" layer="91"/>
@@
 </segment>
 </net>
-<net name="MOSI" class="0">
+<net name="D12" class="0">
 <segment>
 <wire x1="129.54" y1="96.52" x2="134.62" y2="96.52" width="0.1524" layer="91"/>
@@
 </segment>
 </net>
-<net name="!CS" class="0">
+<net name="D10" class="0">
 <segment>
 <wire x1="129.54" y1="93.98" x2="134.62" y2="93.98" width="0.1524" layer="91"/>
@@
 </segment>
 </net>
-<net name="SS2" class="0">
+<net name="D4" class="0">
 <segment>
 <wire x1="129.54" y1="91.44" x2="134.62" y2="91.44" width="0.1524" layer="91"/>
@@
 </segment>
 </net>
-<net name="SS1" class="0">
+<net name="D5" class="0">
 <segment>
 <wire x1="129.54" y1="88.9" x2="134.62" y2="88.9" width="0.1524" layer="91"/>
@@
 </segment>
 </net>
-<net name="IO2" class="0">
+<net name="D2" class="0">
 <segment>
 <wire x1="129.54" y1="86.36" x2="134.62" y2="86.36" width="0.1524" layer="91"/>
@@
 </segment>
 </net>
-<net name="IO1" class="0">
+<net name="D3" class="0">
 <segment>
 <wire x1="129.54" y1="83.82" x2="134.62" y2="83.82" width="0.1524" layer="91"/>
@@
 </segment>
 </net>
-<net name="!IRQ" class="0">
+<net name="A1" class="0">
 <segment>
 <wire x1="129.54" y1="81.28" x2="134.62" y2="81.28" width="0.1524" layer="91"/>
@@
 </segment>
 </net>
-<net name="!RTS" class="0">
+<net name="A6" class="0">
 <segment>
 <wire x1="129.54" y1="76.2" x2="134.62" y2="76.2" width="0.1524" layer="91"/>
@@
 </segment>
 </net>
-<net name="!CTS" class="0">
+<net name="A2" class="0">
 <segment>
 <wire x1="129.54" y1="73.66" x2="134.62" y2="73.66" width="0.1524" layer="91"/>
@@
 </segment>
 </net>
-<net name="!RI" class="0">
+<net name="A9" class="0">
 <segment>
 <wire x1="76.2" y1="76.2" x2="73.66" y2="76.2" width="0.1524" layer="91"/>
@@
 </segment>
 </net>
-<net name="!DCD" class="0">
+<net name="A8" class="0">
 <segment>
 <wire x1="76.2" y1="73.66" x2="73.66" y2="73.66" width="0.1524" layer="91"/>
@@
 </segment>
 </net>
-<net name="!DSR" class="0">
+<net name="A7" class="0">
 <segment>
 <wire x1="76.2" y1="71.12" x2="73.66" y2="71.12" width="0.1524" layer="91"/>
@@
 </segment>
 </net>
-<net name="!DTR" class="0">
+<net name="A3" class="0">
 <segment>
 <wire x1="76.2" y1="68.58" x2="73.66" y2="68.58" width="0.1524" layer="91"/>
@@
 </segment>
 </net>
-<net name="RXD3" class="0">
+<net name="D7" class="0">
 <segment>
 <pinref part="TEENSY" gate="G$1" pin="7"/>
@@
 </segment>
 </net>
-<net name="TXD3" class="0">
+<net name="D8" class="0">
 <segment>
 <pinref part="TEENSY" gate="G$1" pin="8"/>
@@
 </segment>
 </net>
-<net name="RXD1" class="0">
+<net name="D0" class="0">
 <segment>
 <pinref part="TEENSY" gate="G$1" pin="0"/>
@@
 </segment>
 </net>
-<net name="TXD1" class="0">
+<net name="D1" class="0">
 <segment>
 <pinref part="TEENSY" gate="G$1" pin="1"/>
