File: TSOC_Teensy3x/revisions/R2_0/TSOC_Teensy3X.brd (EAGLE design)
At the start: 44.5 x 30.5 mm, 12 parts, among them J1 4P-2.0, J2 4P-2.0

Commit message: update BOM
Parts:
- removed J1, J2: 4P-2.0, Seeed-Connector -2016:HW4-2.0
- added 5V0: (no value), PatternAgents-ProtoPads:WPAD-1-PTH-2.54
- added ANALOG, UART: 4P-2.0-90D, Seeed-Connector -2016:HW4-2.0-90D
- moved GND 14.2 mm to (42.9, 12.7), turned to 90 degrees
- moved FID2 0.80 mm to (42.7, 3.81)
- moved TEENSY 0.76 mm to (26.4, 15.2)
- moved U$1 0.76 mm to (33.5, 16.0)
- moved U$5 0.76 mm to (16.8, 15.7)
- moved FID1 0.25 mm to (2.03, 3.81)
- moved FID3 0.25 mm to (2.03, 26.7)
Connections:
- new net A0: ANALOG.1, TEENSY.14/A0
- new net D9: ANALOG.2, TEENSY.9
- net 3V3: now also ANALOG.3, UART.3; no longer J1.3, J2.3
- net 5V0: now also 5V0.1
- net GND: now also ANALOG.4, UART.4; no longer J1.4, J2.4
- net RXD3: now also UART.1; no longer J2.1
- net SCL: no longer J1.1
- net SDA: no longer J1.2
- net TXD3: now also UART.2; no longer J2.2
Routing:
- net SCL: track 45.1 -> 18.9 mm
- net D9: track 0.00 -> 22.9 mm, vias 0 -> 3
- net SDA: track 28.1 -> 16.4 mm
- net 3V3: track 85.8 -> 97.0 mm, vias 4 -> 3
- net A0: track 0.00 -> 6.73 mm
- net GND: track 99.7 -> 104.0 mm, vias 5 -> 3
- net RXD3: track 22.7 -> 19.5 mm
- net TXD3: track 18.4 -> 15.5 mm
- net 5V0: track 34.0 -> 36.7 mm
- net !IRQ: track 33.5 -> 34.8 mm
- net !CS: track 9.94 -> 8.88 mm
- net MOSI: track 7.40 -> 6.64 mm
Other:
- board text added: "A0"
- board text added: "ANALOG"
- board text added: "D9"
- board text added: "Rev. 2.0"
- board text added: "TSOC_TEENSY3.2"
- board text removed: "I2C"
- board text removed: "Rev. 1.1"
- board text removed: "SCL/ D19"
- board text removed: "SDA/ D18"
