File: TSOC_Teensy3x/revisions/R2_0/TSOC_Teensy3X.sch (EAGLE design)
At the start: 11 parts, among them J1 4P-2.0, J2 4P-2.0

Commit message: update BOM
Parts:
- removed J1, J2: 4P-2.0, Seeed-Connector -2016:GROVE-CONNECTOR-DIP(4P-2.0)
- added 5V0: (no value), PatternAgents-ProtoPads:WPAD-1-PTH
- added ANALOG, UART: 4P-2.0-90D, Seeed-Connector -2016:GROVE-CONNECTOR-DIP-90D(4P-2.0)
Connections:
- new net A0: ANALOG.1, TEENSY.14/A0
- new net D9: ANALOG.2, TEENSY.9
- new net VBAT: TEENSY.VBAT
- net 3V3: now also ANALOG.3, UART.3; no longer J1.3, J2.3
- net 5V0: now also 5V0.1
- net GND: now also ANALOG.4, UART.4; no longer J1.4, J2.4
- net RXD3: now also UART.1; no longer J2.1
- net SCL: no longer J1.1
- net SDA: no longer J1.2
- net TXD3: now also UART.2; no longer J2.2
Other:
- moved on the sheet: GND
Changed lines of the file:
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@@
 <part name="U$2" library="thingSoC" deviceset="TSOC-PCB" device="-SINGLE"/>
 <part name="TSOC" library="thingSoC" deviceset="TSOC-24" device="-BB"/>
-<part name="J1" library="Seeed-Connector -2016" deviceset="GROVE-CONNECTOR-DIP(4P-2.0)" device="" value="4P-2.0"/>
-<part name="J2" library="Seeed-Connector -2016" deviceset="GROVE-CONNECTOR-DIP(4P-2.0)" device="" value="4P-2.0"/>
+<part name="ANALOG" library="Seeed-Connector -2016" deviceset="GROVE-CONNECTOR-DIP-90D(4P-2.0)" device="" value="4P-2.0-90D"/>
+<part name="UART" library="Seeed-Connector -2016" deviceset="GROVE-CONNECTOR-DIP-90D(4P-2.0)" device="" value="4P-2.0-90D"/>
 <part name="FRAME1" library="PatternAgents-Beautify" deviceset="FRAME_ASIZE_LANDSCAPE" device=""/>
 <part name="U$5" library="thingSoC" deviceset="TSOC-LOGO" device="-LRG"/>
@@
 <part name="FID4" library="TSOC-ESP8266-BASE" deviceset="FIDUCIAL" device="UFIDUCIAL"/>
 <part name="FID1" library="TSOC-ESP8266-BASE" deviceset="FIDUCIAL" device="UFIDUCIAL"/>
+<part name="5V0" library="PatternAgents-ProtoPads" deviceset="WPAD-1" device="-PTH"/>
 <part name="GND" library="PatternAgents-ProtoPads" deviceset="WPAD-1" device="-PTH"/>
 </parts>
@@
 <instances>
 <instance part="TEENSY" gate="G$1" x="177.8" y="116.84"/>
-<instance part="U$2" gate="G$1" x="177.8" y="157.48"/>
+<instance part="U$2" gate="G$1" x="154.94" y="25.4"/>
 <instance part="TSOC" gate="TSOC" x="106.68" y="114.3"/>
-<instance part="J1" gate="G$1" x="87.63" y="157.48" rot="R180"/>
-<instance part="J2" gate="G$1" x="118.11" y="157.48" rot="R180"/>
+<instance part="ANALOG" gate="G$1" x="87.63" y="157.48" rot="R180"/>
+<instance part="UART" gate="G$1" x="118.11" y="157.48" rot="R180"/>
 <instance part="FRAME1" gate="G$2" x="172.72" y="0"/>
 <instance part="FRAME1" gate="G$1" x="0" y="0"/>
@@
 <instance part="FID4" gate="G$1" x="264.16" y="27.94"/>
 <instance part="FID1" gate="G$1" x="269.24" y="27.94"/>
-<instance part="GND" gate="G$1" x="170.18" y="172.72" rot="R180"/>
+<instance part="5V0" gate="G$1" x="175.26" y="160.02" rot="R180"/>
+<instance part="GND" gate="G$1" x="175.26" y="149.86" rot="R180"/>
 </instances>
 <busses>
@@
 </segment>
 <segment>
-<pinref part="J1" gate="G$1" pin="4"/>
+<pinref part="ANALOG" gate="G$1" pin="4"/>
 <wire x1="91.44" y1="161.29" x2="97.79" y2="161.29" width="0.1524" layer="91"/>
 <label x="97.79" y="161.29" size="1.016" layer="95" font="vector" ratio="10" xref="yes"/>
 </segment>
 <segment>
-<pinref part="J2" gate="G$1" pin="4"/>
+<pinref part="UART" gate="G$1" pin="4"/>
 <wire x1="121.92" y1="161.29" x2="128.27" y2="161.29" width="0.1524" layer="91"/>
 <label x="128.27" y="161.29" size="1.016" layer="95" font="vector" ratio="10" xref="yes"/>
 </segment>
 <segment>
-<wire x1="175.26" y1="172.72" x2="172.72" y2="172.72" width="0.1524" layer="91"/>
-<label x="180.34" y="172.72" size="1.016" layer="95" font="vector" ratio="10" xref="yes"/>
+<wire x1="180.34" y1="149.86" x2="177.8" y2="149.86" width="0.1524" layer="91"/>
+<label x="185.42" y="149.86" size="1.016" layer="95" font="vector" ratio="10" xref="yes"/>
 <pinref part="GND" gate="G$1" pin="1"/>
-<wire x1="172.72" y1="172.72" x2="180.34" y2="172.72" width="0.1524" layer="91"/>
-<junction x="172.72" y="172.72"/>
+<wire x1="177.8" y1="149.86" x2="185.42" y2="149.86" width="0.1524" layer="91"/>
+<junction x="177.8" y="149.86"/>
 </segment>
 </net>
@@
 <pinref part="TSOC" gate="TSOC" pin="SCL"/>
 </segment>
-<segment>
-<pinref part="J1" gate="G$1" pin="1"/>
-<wire x1="91.44" y1="153.67" x2="97.79" y2="153.67" width="0.1524" layer="91"/>
-<label x="97.79" y="153.67" size="1.016" layer="95" font="vector" ratio="10" xref="yes"/>
-</segment>
 </net>
 <net name="SDA" class="0">
@@
 <pinref part="TSOC" gate="TSOC" pin="SDA"/>
 </segment>
-<segment>
-<pinref part="J1" gate="G$1" pin="2"/>
-<wire x1="91.44" y1="156.21" x2="97.79" y2="156.21" width="0.1524" layer="91"/>
-<label x="97.79" y="156.21" size="1.016" layer="95" font="vector" ratio="10" xref="yes"/>
-</segment>
 </net>
 <net name="SCK" class="0">
@@
 <pinref part="TSOC" gate="TSOC" pin="5V0"/>
 </segment>
+<segment>
+<wire x1="180.34" y1="160.02" x2="177.8" y2="160.02" width="0.1524" layer="91"/>
+<label x="185.42" y="160.02" size="1.016" layer="95" font="vector" ratio="10" xref="yes"/>
+<pinref part="5V0" gate="G$1" pin="1"/>
+<wire x1="177.8" y1="160.02" x2="185.42" y2="160.02" width="0.1524" layer="91"/>
+<junction x="177.8" y="160.02"/>
+</segment>
 </net>
 <net name="3V3" class="0">
@@
 </segment>
 <segment>
-<pinref part="J1" gate="G$1" pin="3"/>
+<pinref part="ANALOG" gate="G$1" pin="3"/>
 <wire x1="91.44" y1="158.75" x2="97.79" y2="158.75" width="0.1524" layer="91"/>
 <label x="97.79" y="158.75" size="1.016" layer="95" font="vector" ratio="10" xref="yes"/>
 </segment>
 <segment>
-<pinref part="J2" gate="G$1" pin="3"/>
+<pinref part="UART" gate="G$1" pin="3"/>
 <wire x1="121.92" y1="158.75" x2="128.27" y2="158.75" width="0.1524" layer="91"/>
 <label x="128.27" y="158.75" size="1.016" layer="95" font="vector" ratio="10" xref="yes"/>
@@
 </segment>
 <segment>
-<pinref part="J2" gate="G$1" pin="1"/>
+<pinref part="UART" gate="G$1" pin="1"/>
 <wire x1="121.92" y1="153.67" x2="128.27" y2="153.67" width="0.1524" layer="91"/>
 <label x="128.27" y="153.67" size="1.016" layer="95" font="vector" ratio="10" xref="yes"/>
@@
 </segment>
 <segment>
-<pinref part="J2" gate="G$1" pin="2"/>
+<pinref part="UART" gate="G$1" pin="2"/>
 <wire x1="121.92" y1="156.21" x2="128.27" y2="156.21" width="0.1524" layer="91"/>
 <label x="128.27" y="156.21" size="1.016" layer="95" font="vector" ratio="10" xref="yes"/>
@@
 </segment>
 </net>
+<net name="A0" class="0">
+<segment>
+<pinref part="TEENSY" gate="G$1" pin="14/A0"/>
+<wire x1="193.04" y1="96.52" x2="198.12" y2="96.52" width="0.1524" layer="91"/>
+<label x="198.12" y="96.52" size="1.016" layer="95" font="vector" ratio="10" xref="yes"/>
+</segment>
+<segment>
+<pinref part="ANALOG" gate="G$1" pin="1"/>
+<wire x1="91.44" y1="153.67" x2="97.79" y2="153.67" width="0.1524" layer="91"/>
+<label x="97.79" y="153.67" size="1.016" layer="95" font="vector" ratio="10" xref="yes"/>
+</segment>
+</net>
+<net name="D9" class="0">
+<segment>
+<pinref part="TEENSY" gate="G$1" pin="9"/>
+<wire x1="162.56" y1="106.68" x2="157.48" y2="106.68" width="0.1524" layer="91"/>
+<label x="157.48" y="106.68" size="1.016" layer="95" font="vector" ratio="10" rot="R180" xref="yes"/>
+</segment>
+<segment>
+<pinref part="ANALOG" gate="G$1" pin="2"/>
+<wire x1="91.44" y1="156.21" x2="97.79" y2="156.21" width="0.1524" layer="91"/>
+<label x="97.79" y="156.21" size="1.016" layer="95" font="vector" ratio="10" xref="yes"/>
+</segment>
+</net>
+<net name="VBAT" class="0">
+<segment>
+<pinref part="TEENSY" gate="G$1" pin="VBAT"/>
+<wire x1="193.04" y1="137.16" x2="203.2" y2="137.16" width="0.1524" layer="91"/>
+<label x="203.2" y="137.16" size="1.016" layer="95" font="vector" ratio="10" xref="yes"/>
+</segment>
+</net>
