File: TSOC_Teensy3x/revisions/R0_2/TSOC_Teensy3X.brd (EAGLE design)
At the start: 44.5 x 30.5 mm, 13 parts

Commit message: update to Rev1.2
Routing:
- net GND: track 104.0 -> 109.1 mm
Other:
- board text added: "UART3"
Changed lines of the file:
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@@
 <text x="40.132" y="10.668" size="0.8128" layer="21" font="vector" ratio="15" rot="R90">Teensy 3.X</text>
 <text x="5.588" y="23.114" size="0.8128" layer="22" font="vector" ratio="15" rot="MR0">GND</text>
-<text x="5.334" y="21.336" size="0.8128" layer="22" font="vector" ratio="15" rot="MR0">3V3</text>
-<text x="5.588" y="18.542" size="0.8128" layer="22" font="vector" ratio="15" rot="MR0">RX3/
+<text x="5.588" y="21.336" size="0.8128" layer="22" font="vector" ratio="15" rot="MR0">3V3</text>
+<text x="5.588" y="16.51" size="0.8128" layer="22" font="vector" ratio="15" rot="MR0">RX3/
 D8</text>
-<text x="5.588" y="16.256" size="0.8128" layer="22" font="vector" ratio="15" rot="MR0">TX3/
+<text x="5.588" y="18.796" size="0.8128" layer="22" font="vector" ratio="15" rot="MR0">TX3/
 D7</text>
-<text x="6.096" y="24.511" size="1.016" layer="22" font="vector" ratio="15" rot="MR0">UART</text>
+<text x="6.096" y="24.511" size="1.016" layer="22" font="vector" ratio="15" rot="MR0">UART3</text>
 <text x="6.858" y="4.699" size="1.016" layer="22" font="vector" ratio="15" rot="MR0">ANALOG</text>
 <text x="5.588" y="12.446" size="0.8128" layer="22" font="vector" ratio="15" rot="MR0">GND</text>
@@
 <contactref element="TSOC" pad="12C"/>
 <polygon width="0.254" layer="1" spacing="0.254" pour="hatch" isolate="0.254" orphans="yes">
-<vertex x="1.016" y="0"/>
-<vertex x="0" y="1.27"/>
+<vertex x="44.45" y="29.21"/>
+<vertex x="44.45" y="1.83161875" curve="-90"/>
+<vertex x="42.61838125" y="0"/>
+<vertex x="0" y="0"/>
 <vertex x="0" y="29.21"/>
 <vertex x="1.016" y="30.48"/>
 <vertex x="43.18" y="30.48"/>
-<vertex x="44.45" y="29.21"/>
-<vertex x="44.45" y="1.524"/>
-<vertex x="42.926" y="0"/>
 </polygon>
 <polygon width="0.254" layer="16" spacing="0.254" pour="hatch" isolate="0.254" orphans="yes">
-<vertex x="1.016" y="0"/>
-<vertex x="0" y="1.27"/>
+<vertex x="44.45" y="29.21"/>
+<vertex x="44.45" y="1.83161875" curve="-90"/>
+<vertex x="42.61838125" y="0"/>
+<vertex x="0" y="0"/>
 <vertex x="0" y="29.21"/>
 <vertex x="1.016" y="30.48"/>
 <vertex x="43.18" y="30.48"/>
-<vertex x="44.45" y="29.21"/>
-<vertex x="44.45" y="1.524"/>
-<vertex x="42.926" y="0"/>
 </polygon>
 <wire x1="9.144" y1="26.67" x2="7.112" y2="26.67" width="0.6096" layer="1"/>
@@
 <wire x1="42.926" y1="22.86" x2="42.926" y2="24.892" width="0.6096" layer="1"/>
 <wire x1="42.926" y1="24.892" x2="42.672" y2="25.146" width="0.6096" layer="1"/>
-<wire x1="42.672" y1="25.146" x2="41.148" y2="25.146" width="0.6096" layer="1"/>
-<wire x1="41.148" y1="25.146" x2="40.894" y2="25.4" width="0.6096" layer="1"/>
+<wire x1="42.672" y1="25.146" x2="40.386" y2="25.146" width="0.6096" layer="1"/>
 <wire x1="40.386" y1="7.62" x2="40.386" y2="12.7" width="0.6096" layer="16"/>
 <wire x1="40.386" y1="12.7" x2="40.386" y2="14.986" width="0.6096" layer="16"/>
@@
 <wire x1="7.112" y1="23.574" x2="4.112" y2="23.574" width="0.6096" layer="1"/>
 <wire x1="4.112" y1="23.574" x2="4.064" y2="23.622" width="0.6096" layer="1"/>
+<wire x1="40.386" y1="25.146" x2="40.132" y2="25.4" width="0.6096" layer="1"/>
+<wire x1="40.132" y1="25.4" x2="40.132" y2="29.718" width="0.6096" layer="1"/>
 </signal>
 <signal name="!ATN">
